Commit message: hillclimber done

File: data/body.urdf (robot description, URDF)
Before this commit: robot robot, 3 links, 2 joints
Joints:
- joint Torso_BackLeg: origin xyz=0.5 0 1 rpy=0 0 0 -> xyz=1.0 0.0 1.0 rpy=0 0 0
- joint Torso_FrontLeg: origin xyz=1.5 0 1 rpy=0 0 0 -> xyz=2.0 0.0 1.0 rpy=0 0 0
